File: ergogen/output/pcbs/hotswap_cuts.kicad_pcb (KiCad board)
At the start: 2 copper layers, 220.4 x 89.6 mm, 37 parts

Commit message: release
Parts:
- GL1, GL10, GL11, GL12, GL13, GL14, GL15, GL16, GL17, GL18, GL19, GL2, GL20, GL21, GL22, GL23, GL24, GL25, GL26, GL27, GL28, GL29, GL3, GL30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: footprint hotswap_cutout -> hotswap_v2_pin_cutout
Other:
- board size 220.4 x 89.6 mm -> 220.4 x 92.6 mm
